File: power_management.kicad_sch (KiCad schematic)
At the start: 38 parts, among them U1 TPS65185

Commit message: Full Schematic
Parts:
- removed R4, R5: 10k, symbol Device:R
Connections:
- net 3.3VIN: now also C3.2, U1.24 (VIN_P); no longer C3.1
- net GND: now also C19.1, C3.1
Other:
- note added: "This schematic is based on the "Typical Application" of the TPS65185 datasheet in Section 9.2. It is suited for the required rails -20V, -15V, 15V, 22V and 3.3V. This schematic assumes a VIN power of 3.3V, that is also used for the pull-up resistors of ~{INT} and PWR_GOOD."
- note removed: "This schematic is based on the "Typical Application" of the TPS65185 datasheet in Section 9.2 It is suited for the required rails -20V, -15V, 15V, 22V and 3.3V"
