File: ED060SC4_SPI_driver_board.kicad_pcb (KiCad board)
At the start: 4 copper layers, 71.2 x 44.5 mm, 86 parts, among them J1 ED060SC4, J2 Conn_01x06, J3 Conn_01x04, J4 Conn_01x04, J5 Conn_01x06, J6 Conn_01x02, SW1 SS12D07VG2, SW2 DSIC01LSGET, U1 TPS65185RGZR, U2 STM32F103C8T6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

Commit message: add JLC order # text for location
Other:
- board text added: "JLCJLCJLCJLC"
Changed lines of the file:
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@@
     (effects (font (size 0.8 0.8) (thickness 0.15) bold) (justify left bottom))
+  )
+  (gr_text "JLCJLCJLCJLC" (at 50.25 65.25 90) (layer "F.SilkS")
+    (effects (font (size 0.8 0.4) (thickness 0.1) bold) (justify left bottom))
   )
   (gr_text "ED060SC4 Driver Board\n" (at 86.75 53.75) (layer "F.SilkS")

Commit message: Add VN pad under TPS and fix some typos
Routing:
- added copper zone on B.Cu, net /EPD Power Rails/VN
Changed lines of the file:
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@@
     (property "ki_keywords" "mounting hole")
     (attr exclude_from_pos_files)
-    (fp_text reference "H1" (at 2 3) (layer "F.SilkS")
+    (fp_text reference "H1" (at 2 3) (layer "F.SilkS") hide
         (effects (font (size 1 1) (thickness 0.15)))
     )
@@
       )
     )
+  )
+  (zone (net 77) (net_name "/EPD Power Rails/VN") (layer "B.Cu") (hatch edge 0.5)
+    (priority 6)
+    (connect_pads yes (clearance 0.5))
+    (min_thickness 0.25) (filled_areas_thickness no)
+    (fill yes (thermal_gap 0.5) (thermal_bridge_width 0.5))
+    (polygon
+      (pts
+        (xy 96 65.75)
+        (xy 103.5 65.75)
+        (xy 103.5 73.25)
+        (xy 96 73.25)
+      )
+    )
